Commit message: change robot morphology to add 4 more dofs

File: world/cube_-10.urdf (robot description, URDF)
Before this commit: robot robot, 1 links, 0 joints
Links:
- link Cube-10: geometry collision box size=1 600 0.22958665930463573; visual box size=1 600 0.22958665930463573

File: world/cube_-11.urdf (robot description, URDF)
Before this commit: robot robot, 1 links, 0 joints
Links:
- link Cube-11: geometry collision box size=1 600 0.044867802522525195; visual box size=1 600 0.044867802522525195

File: world/cube_-12.urdf (robot description, URDF)
Before this commit: robot robot, 1 links, 0 joints
Links:
- link Cube-12: geometry collision box size=1 600 0.08615558355108076; visual box size=1 600 0.08615558355108076

File: world/cube_-13.urdf (robot description, URDF)
Before this commit: robot robot, 1 links, 0 joints
Links:
- link Cube-13: geometry collision box size=1 600 0.050093021712080264; visual box size=1 600 0.050093021712080264

File: world/cube_-14.urdf (robot description, URDF)
Before this commit: robot robot, 1 links, 0 joints
Links:
- link Cube-14: geometry collision box size=1 600 0.25803979977201674; visual box size=1 600 0.25803979977201674

File: world/cube_-15.urdf (robot description, URDF)
Before this commit: robot robot, 1 links, 0 joints
Links:
- link Cube-15: geometry collision box size=1 600 0.1686213702454145; visual box size=1 600 0.1686213702454145

File: world/cube_-16.urdf (robot description, URDF)
Before this commit: robot robot, 1 links, 0 joints
Links:
- link Cube-16: geometry collision box size=1 600 0.21328552352077576; visual box size=1 600 0.21328552352077576

File: world/cube_-17.urdf (robot description, URDF)
Before this commit: robot robot, 1 links, 0 joints
Links:
- link Cube-17: geometry collision box size=1 600 0.10448122868916308; visual box size=1 600 0.10448122868916308

File: world/cube_-18.urdf (robot description, URDF)
Before this commit: robot robot, 1 links, 0 joints
Links:
- link Cube-18: geometry collision box size=1 600 0.025075381860800737; visual box size=1 600 0.025075381860800737

File: world/cube_-19.urdf (robot description, URDF)
Before this commit: robot robot, 1 links, 0 joints
Links:
- link Cube-19: geometry collision box size=1 600 0.017115525713624645; visual box size=1 600 0.017115525713624645

File: world/cube_-2.urdf (robot description, URDF)
Before this commit: robot robot, 1 links, 0 joints
Links:
- link Cube-2: geometry collision box size=1 600 0.1977199503782545; visual box size=1 600 0.1977199503782545

File: world/cube_-20.urdf (robot description, URDF)
Before this commit: robot robot, 1 links, 0 joints
Links:
- link Cube-20: geometry collision box size=1 600 0.18921435709461376; visual box size=1 600 0.18921435709461376

File: world/cube_-21.urdf (robot description, URDF)
Before this commit: robot robot, 1 links, 0 joints
Links:
- link Cube-21: geometry collision box size=1 600 0.18489590312219048; visual box size=1 600 0.18489590312219048

File: world/cube_-22.urdf (robot description, URDF)
Before this commit: robot robot, 1 links, 0 joints
Links:
- link Cube-22: geometry collision box size=1 600 0.24283118960361225; visual box size=1 600 0.24283118960361225

File: world/cube_-23.urdf (robot description, URDF)
Before this commit: robot robot, 1 links, 0 joints
Links:
- link Cube-23: geometry collision box size=1 600 0.07013617217573494; visual box size=1 600 0.07013617217573494

File: world/cube_-24.urdf (robot description, URDF)
Before this commit: robot robot, 1 links, 0 joints
Links:
- link Cube-24: geometry collision box size=1 600 0.17023314834024492; visual box size=1 600 0.17023314834024492

File: world/cube_-3.urdf (robot description, URDF)
Before this commit: robot robot, 1 links, 0 joints
Links:
- link Cube-3: geometry collision box size=1 600 0.08103867643260544; visual box size=1 600 0.08103867643260544

File: world/cube_-4.urdf (robot description, URDF)
Before this commit: robot robot, 1 links, 0 joints
Links:
- link Cube-4: geometry collision box size=1 600 0.1520422510460982; visual box size=1 600 0.1520422510460982

File: world/cube_-5.urdf (robot description, URDF)
Before this commit: robot robot, 1 links, 0 joints
Links:
- link Cube-5: geometry collision box size=1 600 0.22129955698361167; visual box size=1 600 0.22129955698361167

File: world/cube_-6.urdf (robot description, URDF)
Before this commit: robot robot, 1 links, 0 joints
Links:
- link Cube-6: geometry collision box size=1 600 0.18910098211672116; visual box size=1 600 0.18910098211672116
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