Commit message: good periodic behavior

File: best_body.urdf (robot description, URDF)
Before this commit: robot robot, 9 links, 8 joints
Links:
- added link BackLegRot, mass 0.0; collision box size=0 0 0; visual box size=0 0 0
- added link FrontLegRot, mass 0.0; collision box size=0 0 0; visual box size=0 0 0
- added link LeftLegRot, mass 0.0; collision box size=0 0 0; visual box size=0 0 0
- added link RightLegRot, mass 0.0; collision box size=0 0 0; visual box size=0 0 0
- link Torso: mass 10.0 -> 10
Joints:
- removed joint Torso_BackLeg
- removed joint Torso_FrontLeg
- removed joint Torso_LeftLeg
- removed joint Torso_RightLeg
- added joint BackLegRot_BackLeg: type revolute, parent BackLegRot, child BackLeg, origin xyz=0 0 0 rpy=0 0 0, axis 1 0 0, limit lower=-3.14159 upper=3.14159 effort=0.0 velocity=0.0
- added joint FrontLegRot_FrontLeg: type revolute, parent FrontLegRot, child FrontLeg, origin xyz=0.0 0.0 0.0 rpy=0 0 0, axis 0 1 0, limit lower=-3.14159 upper=3.14159 effort=0.0 velocity=0.0
- added joint LeftLegRot_LeftLeg: type revolute, parent LeftLegRot, child LeftLeg, origin xyz=0 0 0 rpy=0 0 0, axis 0 1 0, limit lower=-3.14159 upper=3.14159 effort=0.0 velocity=0.0
- added joint RightLegRot_RightLeg: type revolute, parent RightLegRot, child RightLeg, origin xyz=0 0 0 rpy=0 0 0, axis 0 1 0, limit lower=-3.14159 upper=3.14159 effort=0.0 velocity=0.0
- added joint Torso_BackLegRot: type revolute, parent Torso, child BackLegRot, origin xyz=0 -0.5 1.0 rpy=0 0 0, axis 0 1 0, limit lower=-3.14159 upper=3.14159 effort=0.0 velocity=0.0
- added joint Torso_FrontLegRot: type revolute, parent Torso, child FrontLegRot, origin xyz=0.0 0.5 1.0 rpy=0 0 0, axis 1 0 0, limit lower=-3.14159 upper=3.14159 effort=0.0 velocity=0.0
- added joint Torso_LeftLegRot: type revolute, parent Torso, child LeftLegRot, origin xyz=-0.5 0 1.0 rpy=0 0 0, axis 1 0 0, limit lower=-3.14159 upper=3.14159 effort=0.0 velocity=0.0
- added joint Torso_RightLegRot: type revolute, parent Torso, child RightLegRot, origin xyz=0.5 0 1.0 rpy=0 0 0, axis 1 0 0, limit lower=-3.14159 upper=3.14159 effort=0.0 velocity=0.0

Commit message: working hyperneat

File: best_body.urdf (robot description, URDF)
Before this commit: robot robot, 13 links, 12 joints
Links:
- link Torso: mass 10 -> 3

Commit message: run hyperneat experiments

File: best_body.urdf (robot description, URDF)
Before this commit: robot robot, 13 links, 12 joints
Links:
- link Torso: mass 3 -> 10
